Commit message: added timers to launches and renamed zed links

File: src/urdf_description/urdf/urdf.xacro (robot description, xacro)
@@ -345,5 +345,5 @@
 </link>
 <!-- ZED2 Camera Links -->
-<link name="zed_camera_link">
+<link name="zed2_camera_link">
   <visual>
     <origin xyz="0 0 0" rpy="0 0 1.5708"/>
@@ -373,11 +373,11 @@
 </link>
 <joint name="zed2_imu_joint" type="fixed">
-  <parent link="zed_camera_link"/>
+  <parent link="zed2_camera_link"/>
   <child link="zed2_imu_link"/>
   <origin xyz="0 0 0" rpy="0 0 0"/>
 </joint>
-<joint name="zed_camera_joint" type="fixed">
-  <parent link="base_link"/>
-  <child link="zed_camera_link"/>
+<joint name="zed2_camera_joint" type="fixed">
+  <parent link="base_link"/>
+  <child link="zed2_camera_link"/>
   <!-- Adjust xyz to where your camera sits on the rover -->
   <origin xyz="0.15 0 0.2" rpy="0 0 0"/>

Commit message: got nav2 to be brought up

File: src/urdf_description/urdf/urdf.xacro (robot description, xacro)
@@ -13,5 +13,5 @@
     <origin xyz="0 0 0" rpy="0 0 0"/>
     <geometry>
-      <mesh filename="file://$(find urdf_description)/meshes/base_link.stl" scale="0.001 0.001 0.001"/>
+      <mesh filename="package://urdf_description/meshes/base_link.stl" scale="0.001 0.001 0.001"/>
     </geometry>
     <material name="silver"/>
@@ -20,5 +20,5 @@
     <origin xyz="0 0 0" rpy="0 0 0"/>
     <geometry>
-      <mesh filename="file://$(find urdf_description)/meshes/base_link.stl" scale="0.001 0.001 0.001"/>
+      <mesh filename="package://urdf_description/meshes/base_link.stl" scale="0.001 0.001 0.001"/>
     </geometry>
   </collision>
@@ -33,5 +33,5 @@
     <origin xyz="0.332727 0.312987 0.083488" rpy="0 0 0"/>
     <geometry>
-      <mesh filename="file://$(find urdf_description)/meshes/Wheel_f1_1.stl" scale="0.001 0.001 0.001"/>
+      <mesh filename="package://urdf_description/meshes/Wheel_f1_1.stl" scale="0.001 0.001 0.001"/>
     </geometry>
     <material name="silver"/>
@@ -40,5 +40,5 @@
     <origin xyz="0.332727 0.312987 0.083488" rpy="0 0 0"/>
     <geometry>
-      <mesh filename="file://$(find urdf_description)/meshes/Wheel_f1_1.stl" scale="0.001 0.001 0.001"/>
+      <mesh filename="package://urdf_description/meshes/Wheel_f1_1.stl" scale="0.001 0.001 0.001"/>
     </geometry>
   </collision>
@@ -53,5 +53,5 @@
     <origin xyz="-0.334113 0.312987 0.077759" rpy="0 0 0"/>
     <geometry>
-      <mesh filename="file://$(find urdf_description)/meshes/Wheel_b1_1.stl" scale="0.001 0.001 0.001"/>
+      <mesh filename="package://urdf_description/meshes/Wheel_b1_1.stl" scale="0.001 0.001 0.001"/>
     </geometry>
     <material name="silver"/>
@@ -60,5 +60,5 @@
     <origin xyz="-0.334113 0.312987 0.077759" rpy="0 0 0"/>
     <geometry>
-      <mesh filename="file://$(find urdf_description)/meshes/Wheel_b1_1.stl" scale="0.001 0.001 0.001"/>
+      <mesh filename="package://urdf_description/meshes/Wheel_b1_1.stl" scale="0.001 0.001 0.001"/>
     </geometry>
   </collision>
@@ -73,5 +73,5 @@
     <origin xyz="0.289603 -0.312987 0.183869" rpy="0 0 0"/>
     <geometry>
-      <mesh filename="file://$(find urdf_description)/meshes/Wheel_f2_1.stl" scale="0.001 0.001 0.001"/>
+      <mesh filename="package://urdf_description/meshes/Wheel_f2_1.stl" scale="0.001 0.001 0.001"/>
     </geometry>
     <material name="silver"/>
@@ -80,5 +80,5 @@
     <origin xyz="0.289603 -0.312987 0.183869" rpy="0 0 0"/>
     <geometry>
-      <mesh filename="file://$(find urdf_description)/meshes/Wheel_f2_1.stl" scale="0.001 0.001 0.001"/>
+      <mesh filename="package://urdf_description/meshes/Wheel_f2_1.stl" scale="0.001 0.001 0.001"/>
     </geometry>
   </collision>
@@ -93,5 +93,5 @@
     <origin xyz="-0.331827 -0.312987 0.086997" rpy="0 0 0"/>
     <geometry>
-      <mesh filename="file://$(find urdf_description)/meshes/Wheel_b2_1.stl" scale="0.001 0.001 0.001"/>
+      <mesh filename="package://urdf_description/meshes/Wheel_b2_1.stl" scale="0.001 0.001 0.001"/>
     </geometry>
     <material name="silver"/>
@@ -100,5 +100,5 @@
     <origin xyz="-0.331827 -0.312987 0.086997" rpy="0 0 0"/>
     <geometry>
-      <mesh filename="file://$(find urdf_description)/meshes/Wheel_b2_1.stl" scale="0.001 0.001 0.001"/>
+      <mesh filename="package://urdf_description/meshes/Wheel_b2_1.stl" scale="0.001 0.001 0.001"/>
     </geometry>
   </collision>
@@ -113,5 +113,5 @@
     <origin xyz="-0.0 0.2032 0.0" rpy="0 0 0"/>
     <geometry>
-      <mesh filename="file://$(find urdf_description)/meshes/Suspension_f1_1.stl" scale="0.001 0.001 0.001"/>
+      <mesh filename="package://urdf_description/meshes/Suspension_f1_1.stl" scale="0.001 0.001 0.001"/>
     </geometry>
     <material name="silver"/>
@@ -120,5 +120,5 @@
     <origin xyz="-0.0 0.2032 0.0" rpy="0 0 0"/>
     <geometry>
-      <mesh filename="file://$(find urdf_description)/meshes/Suspension_f1_1.stl" scale="0.001 0.001 0.001"/>
+      <mesh filename="package://urdf_description/meshes/Suspension_f1_1.stl" scale="0.001 0.001 0.001"/>
     </geometry>
   </collision>
@@ -133,5 +133,5 @@
     <origin xyz="-0.0 -0.2032 0.0" rpy="0 0 0"/>
     <geometry>
-      <mesh filename="file://$(find urdf_description)/meshes/Suspension_f2_1.stl" scale="0.001 0.001 0.001"/>
+      <mesh filename="package://urdf_description/meshes/Suspension_f2_1.stl" scale="0.001 0.001 0.001"/>
     </geometry>
     <material name="silver"/>
@@ -140,5 +140,5 @@
     <origin xyz="-0.0 -0.2032 0.0" rpy="0 0 0"/>
     <geometry>
-      <mesh filename="file://$(find urdf_description)/meshes/Suspension_f2_1.stl" scale="0.001 0.001 0.001"/>
+      <mesh filename="package://urdf_description/meshes/Suspension_f2_1.stl" scale="0.001 0.001 0.001"/>
     </geometry>
   </collision>
@@ -153,5 +153,5 @@
     <origin xyz="-0.0 -0.2032 0.0" rpy="0 0 0"/>
     <geometry>
-      <mesh filename="file://$(find urdf_description)/meshes/Suspension_b2_1.stl" scale="0.001 0.001 0.001"/>
+      <mesh filename="package://urdf_description/meshes/Suspension_b2_1.stl" scale="0.001 0.001 0.001"/>
     </geometry>
     <material name="silver"/>
@@ -160,5 +160,5 @@
     <origin xyz="-0.0 -0.2032 0.0" rpy="0 0 0"/>
     <geometry>
-      <mesh filename="file://$(find urdf_description)/meshes/Suspension_b2_1.stl" scale="0.001 0.001 0.001"/>
+      <mesh filename="package://urdf_description/meshes/Suspension_b2_1.stl" scale="0.001 0.001 0.001"/>
     </geometry>
   </collision>
@@ -173,5 +173,5 @@
     <origin xyz="-0.0 0.2032 0.0" rpy="0 0 0"/>
     <geometry>
-      <mesh filename="file://$(find urdf_description)/meshes/Suspension_b1_1.stl" scale="0.001 0.001 0.001"/>
+      <mesh filename="package://urdf_description/meshes/Suspension_b1_1.stl" scale="0.001 0.001 0.001"/>
     </geometry>
     <material name="silver"/>
@@ -180,5 +180,5 @@
     <origin xyz="-0.0 0.2032 0.0" rpy="0 0 0"/>
     <geometry>
-      <mesh filename="file://$(find urdf_description)/meshes/Suspension_b1_1.stl" scale="0.001 0.001 0.001"/>
+      <mesh filename="package://urdf_description/meshes/Suspension_b1_1.stl" scale="0.001 0.001 0.001"/>
     </geometry>
   </collision>
@@ -193,5 +193,5 @@
     <origin xyz="-0.094063 0.223274 0.016277" rpy="0 0 0"/>
     <geometry>
-      <mesh filename="file://$(find urdf_description)/meshes/4InchRod_b1_1.stl" scale="0.001 0.001 0.001"/>
+      <mesh filename="package://urdf_description/meshes/4InchRod_b1_1.stl" scale="0.001 0.001 0.001"/>
     </geometry>
     <material name="silver"/>
@@ -200,5 +200,5 @@
     <origin xyz="-0.094063 0.223274 0.016277" rpy="0 0 0"/>
     <geometry>
-      <mesh filename="file://$(find urdf_description)/meshes/4InchRod_b1_1.stl" scale="0.001 0.001 0.001"/>
+      <mesh filename="package://urdf_description/meshes/4InchRod_b1_1.stl" scale="0.001 0.001 0.001"/>
     </geometry>
   </collision>
@@ -213,5 +213,5 @@
     <origin xyz="-0.308737 0.289862 -0.048001" rpy="0 0 0"/>
     <geometry>
-      <mesh filename="file://$(find urdf_description)/meshes/4InchBase_b1_1.stl" scale="0.001 0.001 0.001"/>
+      <mesh filename="package://urdf_description/meshes/4InchBase_b1_1.stl" scale="0.001 0.001 0.001"/>
     </geometry>
     <material name="silver"/>
@@ -220,5 +220,5 @@
     <origin xyz="-0.308737 0.289862 -0.048001" rpy="0 0 0"/>
     <geometry>
-      <mesh filename="file://$(find urdf_description)/meshes/4InchBase_b1_1.stl" scale="0.001 0.001 0.001"/>
+      <mesh filename="package://urdf_description/meshes/4InchBase_b1_1.stl" scale="0.001 0.001 0.001"/>
     </geometry>
   </collision>
@@ -233,5 +233,5 @@
     <origin xyz="0.09377 0.229624 0.017891" rpy="0 0 0"/>
     <geometry>
-      <mesh filename="file://$(find urdf_description)/meshes/4InchRod_f1_1.stl" scale="0.001 0.001 0.001"/>
+      <mesh filename="package://urdf_description/meshes/4InchRod_f1_1.stl" scale="0.001 0.001 0.001"/>
     </geometry>
     <material name="silver"/>
@@ -240,5 +240,5 @@
     <origin xyz="0.09377 0.229624 0.017891" rpy="0 0 0"/>
     <geometry>
-      <mesh filename="file://$(find urdf_description)/meshes/4InchRod_f1_1.stl" scale="0.001 0.001 0.001"/>
+      <mesh filename="package://urdf_description/meshes/4InchRod_f1_1.stl" scale="0.001 0.001 0.001"/>
     </geometry>
   </collision>
@@ -253,5 +253,5 @@
     <origin xyz="-0.135311 0.162949 0.043883" rpy="0 0 0"/>
     <geometry>
-      <mesh filename="file://$(find urdf_description)/meshes/4InchBase_f1_1.stl" scale="0.001 0.001 0.001"/>
+      <mesh filename="package://urdf_description/meshes/4InchBase_f1_1.stl" scale="0.001 0.001 0.001"/>
     </geometry>
     <material name="silver"/>
@@ -260,5 +260,5 @@
     <origin xyz="-0.135311 0.162949 0.043883" rpy="0 0 0"/>
     <geometry>
-      <mesh filename="file://$(find urdf_description)/meshes/4InchBase_f1_1.stl" scale="0.001 0.001 0.001"/>
+      <mesh filename="package://urdf_description/meshes/4InchBase_f1_1.stl" scale="0.001 0.001 0.001"/>
     </geometry>
   </collision>
@@ -273,5 +273,5 @@
     <origin xyz="0.272521 -0.071653 -0.358369" rpy="0 0 0"/>
     <geometry>
-      <mesh filename="file://$(find urdf_description)/meshes/4InchBase_f2_1.stl" scale="0.001 0.001 0.001"/>
+      <mesh filename="package://urdf_description/meshes/4InchBase_f2_1.stl" scale="0.001 0.001 0.001"/>
     </geometry>
     <material name="silver"/>
@@ -280,5 +280,5 @@
     <origin xyz="0.272521 -0.071653 -0.358369" rpy="0 0 0"/>
     <geometry>
-      <mesh filename="file://$(find urdf_description)/meshes/4InchBase_f2_1.stl" scale="0.001 0.001 0.001"/>
+      <mesh filename="package://urdf_description/meshes/4InchBase_f2_1.stl" scale="0.001 0.001 0.001"/>
     </geometry>
   </collision>
@@ -293,5 +293,5 @@
     <origin xyz="0.083389 -0.229624 0.046467" rpy="0 0 0"/>
     <geometry>
-      <mesh filename="file://$(find urdf_description)/meshes/4InchRod_f2_1.stl" scale="0.001 0.001 0.001"/>
+      <mesh filename="package://urdf_description/meshes/4InchRod_f2_1.stl" scale="0.001 0.001 0.001"/>
     </geometry>
     <material name="silver"/>
@@ -300,5 +300,5 @@
     <origin xyz="0.083389 -0.229624 0.046467" rpy="0 0 0"/>
     <geometry>
-      <mesh filename="file://$(find urdf_description)/meshes/4InchRod_f2_1.stl" scale="0.001 0.001 0.001"/>
+      <mesh filename="package://urdf_description/meshes/4InchRod_f2_1.stl" scale="0.001 0.001 0.001"/>
     </geometry>
   </collision>
@@ -313,5 +313,5 @@
     <origin xyz="0.170921 -0.071653 -0.358369" rpy="0 0 0"/>
     <geometry>
-      <mesh filename="file://$(find urdf_description)/meshes/4InchBase_b2_1.stl" scale="0.001 0.001 0.001"/>
+      <mesh filename="package://urdf_description/meshes/4InchBase_b2_1.stl" scale="0.001 0.001 0.001"/>
     </geometry>
     <material name="silver"/>
@@ -320,5 +320,5 @@
     <origin xyz="0.170921 -0.071653 -0.358369" rpy="0 0 0"/>
     <geometry>
-      <mesh filename="file://$(find urdf_description)/meshes/4InchBase_b2_1.stl" scale="0.001 0.001 0.001"/>
+      <mesh filename="package://urdf_description/meshes/4InchBase_b2_1.stl" scale="0.001 0.001 0.001"/>
     </geometry>
   </collision>
@@ -333,5 +333,5 @@
     <origin xyz="-0.286268 -0.312144 -0.190441" rpy="0 0 0"/>
     <geometry>
-      <mesh filename="file://$(find urdf_description)/meshes/4InchRod_b2_1.stl" scale="0.001 0.001 0.001"/>
+      <mesh filename="package://urdf_description/meshes/4InchRod_b2_1.stl" scale="0.001 0.001 0.001"/>
     </geometry>
     <material name="silver"/>
@@ -340,5 +340,5 @@
     <origin xyz="-0.286268 -0.312144 -0.190441" rpy="0 0 0"/>
     <geometry>
-      <mesh filename="file://$(find urdf_description)/meshes/4InchRod_b2_1.stl" scale="0.001 0.001 0.001"/>
+      <mesh filename="package://urdf_description/meshes/4InchRod_b2_1.stl" scale="0.001 0.001 0.001"/>
     </geometry>
   </collision>
